Commit message: add file 4 wheel and conclusion

File: src/articubot_one/description/robot_core.xacro (robot description, xacro)
@@ -13,7 +13,13 @@
         <color rgba="0 0 0 1"/>
     </material>
- <material name="red">
-     <color rgba="1 0 0 1"/>
- </material>
+    <material name="red">
+        <color rgba="1 0 0 1"/>
+    </material>
+    <material name="green">
+        <color rgba="0 1 0 1" />
+    </material>
+    <material name="gray">
+        <color rgba="0.5 0.5 0.5 1" />
+    </material>
     <!-- BASE LINK -->
     <link name="base_link">
@@ -22,9 +28,9 @@
         <parent link="base_link"/>
         <child link="chassis"/>
-        <origin xyz="-0.1 0 0"/>
+        <origin xyz="0 0 0"/>
     </joint>
     <link name="chassis">
         <visual>
-            <origin xyz="0.15 0 0.075" rpy="0 0 0"/>
+            <origin xyz="0 0 0.075" rpy="0 0 0"/>
             <geometry>
                 <box size="0.3 0.3 0.15"/>
@@ -33,5 +39,5 @@
         </visual>
         <collision>
-            <origin xyz="0.15 0 0.075" rpy="0 0 0"/>
+            <origin xyz="0 0 0.075" rpy="0 0 0"/>
             <geometry>
                 <box size="0.3 0.3 0.15"/>
@@ -39,33 +45,15 @@
         </collision>
         <xacro:inertial_box mass="0.5" x="0.3" y="0.3" z="0.15">
-            <origin xyz="0.15 0 0.075" rpy="0 0 0"/>
+            <origin xyz="0 0 0.075" rpy="0 0 0"/>
         </xacro:inertial_box>
     </link>
-    <!-- LEFT WHEEL -->
-    <joint name="left_wheel_joint" type="continuous">
+    <!-- FRONT LEFT WHEEL -->
+    <joint name="front_left_wheel_joint" type="continuous">
         <parent link="base_link"/>
-        <child link="left_wheel"/>
-        <origin xyz="0 0.175 0" rpy="-${pi/2} 0 0"/>
+        <child link="front_left_wheel"/>
+        <origin xyz="0.1 0.175 0" rpy="-${pi/2} 0 0"/>
         <axis xyz="0 0 1"/>
     </joint>
-    <link name="left_wheel">
-        <visual>
-            <geometry>
-                <cylinder length="0.04" radius="0.05" />/>
-            </geometry>
-            <material name="blue"/>
-        </visual>
-        <xacro:inertial_cylinder mass="0.1" length="0.05" radius="0.05">
-            <origin xyz="0 0 0" rpy="0 0 0"/>
-        </xacro:inertial_cylinder>
-    </link>
-    <!-- RIGHT WHEEL -->
-    <joint name="right_wheel_joint" type="continuous">
-        <parent link="base_link"/>
-        <child link="right_wheel"/>
-        <origin xyz="0 -0.175 0" rpy="${pi/2} 0 0"/>
-        <axis xyz="0 0 -1"/>
-    </joint>
-    <link name="right_wheel">
+    <link name="front_left_wheel">
         <visual>
             <geometry>
@@ -74,24 +62,81 @@
             <material name="blue"/>
         </visual>
+        <collision>
+            <geometry>
+                <cylinder length="0.04" radius="0.05" />
+            </geometry>
+        </collision>
         <xacro:inertial_cylinder mass="0.1" length="0.05" radius="0.05">
             <origin xyz="0 0 0" rpy="0 0 0"/>
         </xacro:inertial_cylinder>
     </link>
-    <!-- CASTER WHEEL -->
-    <joint name="caster_wheel_joint" type="fixed">
-        <parent link="chassis"/>
-        <child link="caster_wheel"/>
-        <origin xyz="0.24 0 0" rpy="0 0 0"/>
+    <!-- FRONT RIGHT WHEEL -->
+    <joint name="front_right_wheel_joint" type="continuous">
+        <parent link="base_link"/>
+        <child link="front_right_wheel_joint"/>
+        <origin xyz="0.1 -0.175 0" rpy="${pi/2} 0 0"/>
+        <axis xyz="0 0 -1"/>
     </joint>
-    <link name="caster_wheel">
+    <link name="front_right_wheel_joint">
         <visual>
             <geometry>
-                <sphere radius="0.05" />
+                <cylinder length="0.04" radius="0.05" />
             </geometry>
-            <material name="black"/>
+            <material name="red"/>
         </visual>
-        <xacro:inertial_sphere mass="0.1" radius="0.05">
+        <collision>
+            <geometry>
+                <cylinder length="0.04" radius="0.05" />
+            </geometry>
+        </collision>
+        <xacro:inertial_cylinder mass="0.1" length="0.05" radius="0.05">
             <origin xyz="0 0 0" rpy="0 0 0"/>
-        </xacro:inertial_sphere>
+        </xacro:inertial_cylinder>
+    </link>
+    <!-- BACK LEFT WHEEL -->
+    <joint name="back_left_wheel_joint" type="continuous">
+        <parent link="base_link"/>
+        <child link="back_left_wheel"/>
+        <origin xyz="-0.1 0.175 0" rpy="-${pi/2} 0 0"/>
+        <axis xyz="0 0 1"/>
+    </joint>
+    <link name="back_left_wheel">
+        <visual>
+            <geometry>
+                <cylinder length="0.04" radius="0.05" />
+            </geometry>
+            <material name="gray"/>
+        </visual>
+        <collision>
+            <geometry>
+                <cylinder length="0.04" radius="0.05" />
+            </geometry>
+        </collision>
+        <xacro:inertial_cylinder mass="0.1" length="0.05" radius="0.05">
+            <origin xyz="0 0 0" rpy="0 0 0"/>
+        </xacro:inertial_cylinder>
+    </link>
+    <!-- BACK RIGHT WHEEL -->
+    <joint name="back_right_wheel_joint" type="continuous">
+        <parent link="base_link"/>
+        <child link="back_right_wheel_joint"/>
+        <origin xyz="-0.1 -0.175 0" rpy="${pi/2} 0 0"/>
+        <axis xyz="0 0 -1"/>
+    </joint>
+    <link name="back_right_wheel_joint">
+        <visual>
+            <geometry>
+                <cylinder length="0.04" radius="0.05" />
+            </geometry>
+            <material name="green"/>
+        </visual>
+        <collision>
+            <geometry>
+                <cylinder length="0.04" radius="0.05" />
+            </geometry>
+        </collision>
+        <xacro:inertial_cylinder mass="0.1" length="0.05" radius="0.05">
+            <origin xyz="0 0 0" rpy="0 0 0"/>
+        </xacro:inertial_cylinder>
     </link>
 </robot>

Commit message: update gazebo

File: src/articubot_one/description/robot_core.xacro (robot description, xacro)
@@ -21,4 +21,7 @@
     <material name="gray">
         <color rgba="0.5 0.5 0.5 1" />
+    </material>
+    <material name="pink">
+        <color rgba="1 0.4 0.7 1" />
     </material>
     <!-- BASE LINK -->
@@ -48,4 +51,7 @@
         </xacro:inertial_box>
     </link>
+    <gazebo reference="chassis">
+        <material>Gazebo/White</material>
+    </gazebo>
     <!-- FRONT LEFT WHEEL -->
     <joint name="front_left_wheel_joint" type="continuous">
@@ -71,12 +77,15 @@
         </xacro:inertial_cylinder>
     </link>
+    <gazebo reference="front_left_wheel">
+        <material>Gazebo/Blue</material>
+    </gazebo>
     <!-- FRONT RIGHT WHEEL -->
     <joint name="front_right_wheel_joint" type="continuous">
         <parent link="base_link"/>
-        <child link="front_right_wheel_joint"/>
+        <child link="front_right_wheel"/>
         <origin xyz="0.1 -0.175 0" rpy="${pi/2} 0 0"/>
         <axis xyz="0 0 -1"/>
     </joint>
-    <link name="front_right_wheel_joint">
+    <link name="front_right_wheel">
         <visual>
             <geometry>
@@ -94,4 +103,7 @@
         </xacro:inertial_cylinder>
     </link>
+    <gazebo reference="front_right_wheel">
+        <material>Gazebo/Red</material>
+    </gazebo>
     <!-- BACK LEFT WHEEL -->
     <joint name="back_left_wheel_joint" type="continuous">
@@ -117,12 +129,15 @@
         </xacro:inertial_cylinder>
     </link>
+    <gazebo reference="back_left_wheel">
+        <material>Gazebo/Gray</material>
+    </gazebo>
     <!-- BACK RIGHT WHEEL -->
     <joint name="back_right_wheel_joint" type="continuous">
         <parent link="base_link"/>
-        <child link="back_right_wheel_joint"/>
+        <child link="back_right_wheel"/>
         <origin xyz="-0.1 -0.175 0" rpy="${pi/2} 0 0"/>
         <axis xyz="0 0 -1"/>
     </joint>
-    <link name="back_right_wheel_joint">
+    <link name="back_right_wheel">
         <visual>
             <geometry>
@@ -140,3 +155,6 @@
         </xacro:inertial_cylinder>
     </link>
+    <gazebo reference="back_left_wheel">
+        <material>Gazebo/Green</material>
+    </gazebo>
 </robot>
