Commit message: update

File: src/articubot_one/description/inclass_robot_core.xacro (robot description, xacro)
@@ -42,4 +42,7 @@
         </xacro:inertial_box>
     </link>
+    <gazebo reference="chassis">
+        <material>Gazebo/White</material>
+    </gazebo>
     <!-- LEFT WHEEL -->
     <joint name="left_wheel_joint" type="continuous">
@@ -52,5 +55,5 @@
         <visual>
             <geometry>
-                <cylinder length="0.04" radius="0.05" />/>
+                <cylinder length="0.04" radius="0.05" />
             </geometry>
             <material name="blue"/>
@@ -58,5 +61,5 @@
         <collision>
             <geometry>
-                <cylinder length="0.04" radius="0.05" />/>
+                <cylinder length="0.04" radius="0.05" />
             </geometry>
         </collision>
@@ -65,4 +68,7 @@
         </xacro:inertial_cylinder>
     </link>
+    <gazebo reference="left_wheel">
+        <material>Gazebo/Blue</material>
+    </gazebo>
     <!-- RIGHT WHEEL -->
     <joint name="right_wheel_joint" type="continuous">
@@ -81,5 +87,5 @@
         <collision>
             <geometry>
-                <cylinder length="0.04" radius="0.05" />/>
+                <cylinder length="0.04" radius="0.05" />
             </geometry>
         </collision>
@@ -88,4 +94,7 @@
         </xacro:inertial_cylinder>
     </link>
+    <gazebo reference="right_wheel">
+        <material>Gazebo/Blue</material>
+    </gazebo>
     <!-- CASTER WHEEL -->
     <joint name="caster_wheel_joint" type="fixed">
@@ -110,3 +119,8 @@
         </xacro:inertial_sphere>
     </link>
+    <gazebo reference="caster_wheel">
+        <material>Gazebo/Black</material>
+        <mu1 value="0.5"/>
+        <mu2 value="0.5"/>
+    </gazebo>
 </robot>

File: src/articubot_one/description/robot.urdf.xacro (robot description, xacro)
@@ -3,3 +3,6 @@
     <xacro:include filename="inertial_macros.xacro" />
     <xacro:include filename="robot_core.xacro" />
+    <!-- <xacro:include filename="inclass_robot_core.xacro" /> -->
+    <xacro:include filename="gazebo_control.xacro" />
+    <!-- <xacro:include filename="inclass_gazebo_control.xacro" /> -->
 </robot>

Commit message: update slam

File: src/articubot_one/description/inclass_robot_core.xacro (robot description, xacro)
@@ -24,4 +24,12 @@
         <origin xyz="-0.1 0 0"/>
     </joint>
+    <!-- BASE_FOOTPRINT LINK -->
+    <joint name="base_footprint_joint" type="fixed">
+        <parent link="base_link"/>
+        <child link="base_footprint"/>
+        <origin xyz="0 0 0" rpy="0 0 0"/>
+    </joint>
+    <link name="base_footprint">
+    </link>
     <link name="chassis">
         <visual>

File: src/articubot_one/description/robot_core.xacro (robot description, xacro)
@@ -27,4 +27,12 @@
     <!-- BASE LINK -->
     <link name="base_link">
+    </link>
+    <!-- BASE_FOOTPRINT LINK -->
+    <joint name="base_footprint_joint" type="fixed">
+        <parent link="base_link"/>
+        <child link="base_footprint"/>
+        <origin xyz="0 0 0" rpy="0 0 0"/>
+    </joint>
+    <link name="base_footprint">
     </link>
     <joint name="chassis_joint" type="fixed">
