Commit message: add map project

File: src/articubot_one/description/gazebo_control.xacro (robot description, xacro)
@@ -1,23 +1,24 @@
-<?xml version="1.0"?>
-<robot xmlns:xacro="http://www.ros.org/wiki/xacro">
-    <gazebo>
-        <plugin name='diff_drive' filename='libgazebo_ros_diff_drive.so'>
-            <!-- Wheel Information -->
-            <!-- <left_joint>front_left_wheel_joint</left_joint> -->
-            <!-- <right_joint>front_right_wheel_joint</right_joint> -->
-            <left_joint>back_left_wheel_joint</left_joint>
-            <right_joint>back_right_wheel_joint</right_joint>
-            <wheel_separation>0.35</wheel_separation>  <!-- Distance between wheels (update if needed) -->
-            <wheel_diameter>0.1</wheel_diameter>        <!-- Diameter of the wheels (update if needed) -->
-            <!-- Limits -->
-            <max_wheel_torque>200</max_wheel_torque>
-            <max_wheel_acceleration>10.0</max_wheel_acceleration>
-            <!-- Output -->
-            <odometry_frame>odom</odometry_frame>
-            <robot_base_frame>base_link</robot_base_frame>
-            <publish_odom>true</publish_odom>
-            <publish_odom_tf>true</publish_odom_tf>
-            <publish_wheel_tf>true</publish_wheel_tf>
-        </plugin>
-    </gazebo>
-</robot>
+<gazebo>
+    <plugin name="skid_steer_drive_controller" filename="libgazebo_ros_skid_steer_drive.so">
+        <!-- Front Left and Right Wheels -->
+        <leftFrontJoint>front_left_wheel_joint</leftFrontJoint>
+        <rightFrontJoint>front_right_wheel_joint</rightFrontJoint>
+        <!-- Rear Left and Right Wheels -->
+        <leftRearJoint>back_left_wheel_joint</leftRearJoint>
+        <rightRearJoint>back_right_wheel_joint</rightRearJoint>
+        <!-- Skid-steering parameters -->
+        <wheel_separation>0.35</wheel_separation>
+        <wheel_diameter>0.1</wheel_diameter>
+        <!-- Control parameters -->
+        <max_wheel_torque>200</max_wheel_torque>
+        <max_wheel_acceleration>10.0</max_wheel_acceleration>
+        <!-- Odometry configuration -->
+        <odometry_frame>odom</odometry_frame>
+        <robot_base_frame>base_link</robot_base_frame>
+        <publish_odom>true</publish_odom>
+        <publish_odom_tf>true</publish_odom_tf>
+        <publish_wheel_tf>true</publish_wheel_tf>
+        <!-- Four-wheel drive control -->
+        <use_4wd>true</use_4wd>
+    </plugin>
+</gazebo>

File: src/articubot_one/description/inclass_robot_core.xacro (robot description, xacro)
@@ -19,9 +19,4 @@
     <link name="base_link">
     </link>
-    <joint name="chassis_joint" type="fixed">
-        <parent link="base_link"/>
-        <child link="chassis"/>
-        <origin xyz="-0.1 0 0"/>
-    </joint>
     <!-- BASE_FOOTPRINT LINK -->
     <joint name="base_footprint_joint" type="fixed">
@@ -32,4 +27,9 @@
     <link name="base_footprint">
     </link>
+    <joint name="chassis_joint" type="fixed">
+        <parent link="base_link"/>
+        <child link="chassis"/>
+        <origin xyz="-0.1 0 0"/>
+    </joint>
     <link name="chassis">
         <visual>

File: src/articubot_one/description/robot_core.xacro (robot description, xacro)
@@ -126,5 +126,5 @@
                 <cylinder length="0.04" radius="0.05" />
             </geometry>
-            <material name="gray"/>
+            <material name="orange"/>
         </visual>
         <collision>
@@ -138,5 +138,5 @@
     </link>
     <gazebo reference="back_left_wheel">
-        <material>Gazebo/Gray</material>
+        <material>Gazebo/Orange</material>
     </gazebo>
     <!-- BACK RIGHT WHEEL -->

Commit message: modify robot and add box  to map and change map color

File: src/articubot_one/description/gazebo_control.xacro (robot description, xacro)
@@ -1,24 +1,37 @@
-<gazebo>
-    <plugin name="skid_steer_drive_controller" filename="libgazebo_ros_skid_steer_drive.so">
-        <!-- Front Left and Right Wheels -->
-        <leftFrontJoint>front_left_wheel_joint</leftFrontJoint>
-        <rightFrontJoint>front_right_wheel_joint</rightFrontJoint>
-        <!-- Rear Left and Right Wheels -->
-        <leftRearJoint>back_left_wheel_joint</leftRearJoint>
-        <rightRearJoint>back_right_wheel_joint</rightRearJoint>
-        <!-- Skid-steering parameters -->
-        <wheel_separation>0.35</wheel_separation>
-        <wheel_diameter>0.1</wheel_diameter>
-        <!-- Control parameters -->
-        <max_wheel_torque>200</max_wheel_torque>
-        <max_wheel_acceleration>10.0</max_wheel_acceleration>
-        <!-- Odometry configuration -->
-        <odometry_frame>odom</odometry_frame>
-        <robot_base_frame>base_link</robot_base_frame>
-        <publish_odom>true</publish_odom>
-        <publish_odom_tf>true</publish_odom_tf>
-        <publish_wheel_tf>true</publish_wheel_tf>
-        <!-- Four-wheel drive control -->
-        <use_4wd>true</use_4wd>
-    </plugin>
-</gazebo>
+<?xml version="1.0"?>
+<robot xmlns:xacro="http://www.ros.org/wiki/xacro">
+    <gazebo>
+        <plugin name='back_wheel' filename='libgazebo_ros_diff_drive.so'>
+            <!-- Wheel Information -->
+            <left_joint>back_left_wheel_joint</left_joint>
+            <right_joint>back_right_wheel_joint</right_joint>
+            <wheel_separation>0.35</wheel_separation>
+            <wheel_diameter>0.1</wheel_diameter>
+            <!-- Limits -->
+            <max_wheel_torque>200</max_wheel_torque>
+            <max_wheel_acceleration>10.0</max_wheel_acceleration>
+            <!-- Output -->
+            <odometry_frame>odom</odometry_frame>
+            <robot_base_frame>base_link</robot_base_frame>
+            <publish_odom>true</publish_odom>
+            <publish_odom_tf>true</publish_odom_tf>
+            <publish_wheel_tf>true</publish_wheel_tf>
+        </plugin>
+        <plugin name='front_wheel' filename='libgazebo_ros_diff_drive.so'>
+            <!-- Wheel Information -->
+            <left_joint>front_left_wheel_joint</left_joint>
+            <right_joint>front_right_wheel_joint</right_joint>
+            <wheel_separation>0.35</wheel_separation>
+            <wheel_diameter>0.1</wheel_diameter>
+            <!-- Limits -->
+            <max_wheel_torque>200</max_wheel_torque>
+            <max_wheel_acceleration>10.0</max_wheel_acceleration>
+            <!-- Output -->
+            <odometry_frame>odom</odometry_frame>
+            <robot_base_frame>base_link</robot_base_frame>
+            <publish_odom>true</publish_odom>
+            <publish_odom_tf>true</publish_odom_tf>
+            <publish_wheel_tf>true</publish_wheel_tf>
+        </plugin>
+    </gazebo>
+</robot>

File: src/articubot_one/description/lidar.xacro (robot description, xacro)
@@ -4,5 +4,5 @@
         <parent link="chassis"/>
         <child link="laser_frame"/>
-        <origin xyz="0 0 0.155" rpy="0 0 0"/>
+        <origin xyz="0 0 0.215" rpy="0 0 0"/>
     </joint>
     <link name="laser_frame">
@@ -26,5 +26,5 @@
         <sensor name="laser" type="ray">
             <pose> 0 0 0 0 0 0 </pose>
-            <visualize>true</visualize>
+            <visualize>false</visualize>
             <update_rate>10</update_rate>
             <ray>

File: src/articubot_one/description/robot.urdf.xacro (robot description, xacro)
@@ -3,6 +3,6 @@
     <xacro:include filename="inertial_macros.xacro" />
     <xacro:include filename="robot_core.xacro" />
+    <xacro:include filename="gazebo_control.xacro" />
     <!-- <xacro:include filename="inclass_robot_core.xacro" /> -->
-    <xacro:include filename="gazebo_control.xacro" />
     <!-- <xacro:include filename="inclass_gazebo_control.xacro" /> -->
     <xacro:include filename="lidar.xacro" />

File: src/articubot_one/description/robot_core.xacro (robot description, xacro)
@@ -41,20 +41,25 @@
         <origin xyz="0 0 0"/>
     </joint>
+    <!-- Chassis Link -->
     <link name="chassis">
         <visual>
-            <origin xyz="0 0 0.075" rpy="0 0 0"/>
+            <origin xyz="0 0 0.13" rpy="0 0 0"/>
             <geometry>
-                <box size="0.3 0.3 0.15"/>
+                <box size="0.451 0.451 0.15"/>
+                <!-- Hole geometry -->
+                <cylinder length="0.15" radius="0.075"/>
             </geometry>
             <material name="white"/>
         </visual>
         <collision>
-            <origin xyz="0 0 0.075" rpy="0 0 0"/>
+            <origin xyz="0 0 0.13" rpy="0 0 0"/>
             <geometry>
-                <box size="0.3 0.3 0.15"/>
+                <box size="0.451 0.451 0.15"/>
+                <!-- Hole geometry -->
+                <cylinder length="0.15" radius="0.075"/>
             </geometry>
         </collision>
-        <xacro:inertial_box mass="0.5" x="0.3" y="0.3" z="0.15">
-            <origin xyz="0 0 0.075" rpy="0 0 0"/>
+        <xacro:inertial_box mass="0.5" x="0.451" y="0.451" z="0.15">
+            <origin xyz="0 0 0.13" rpy="0 0 0"/>
         </xacro:inertial_box>
     </link>
@@ -62,15 +67,9 @@
         <material>Gazebo/White</material>
     </gazebo>
-    <!-- FRONT LEFT WHEEL -->
-    <joint name="front_left_wheel_joint" type="continuous">
-        <parent link="base_link"/>
-        <child link="front_left_wheel"/>
-        <origin xyz="0.1 0.175 0" rpy="-${pi/2} 0 0"/>
-        <axis xyz="0 0 1"/>
-    </joint>
+    <!-- Wheel Link -->
     <link name="front_left_wheel">
         <visual>
             <geometry>
-                <cylinder length="0.04" radius="0.05" />
+                <cylinder length="0.03" radius="0.07" />
             </geometry>
             <material name="blue"/>
@@ -78,8 +77,8 @@
         <collision>
             <geometry>
-                <cylinder length="0.04" radius="0.05" />
+                <cylinder length="0.03" radius="0.07" />
             </geometry>
         </collision>
-        <xacro:inertial_cylinder mass="0.1" length="0.05" radius="0.05">
+        <xacro:inertial_cylinder mass="0.1" length="0.03" radius="0.07">
             <origin xyz="0 0 0" rpy="0 0 0"/>
         </xacro:inertial_cylinder>
@@ -88,15 +87,8 @@
         <material>Gazebo/Blue</material>
     </gazebo>
-    <!-- FRONT RIGHT WHEEL -->
-    <joint name="front_right_wheel_joint" type="continuous">
-        <parent link="base_link"/>
-        <child link="front_right_wheel"/>
-        <origin xyz="0.1 -0.175 0" rpy="${pi/2} 0 0"/>
-        <axis xyz="0 0 -1"/>
-    </joint>
     <link name="front_right_wheel">
         <visual>
             <geometry>
-                <cylinder length="0.04" radius="0.05" />
+                <cylinder length="0.03" radius="0.07" />
             </geometry>
             <material name="red"/>
@@ -104,8 +96,8 @@
         <collision>
             <geometry>
-                <cylinder length="0.04" radius="0.05" />
+                <cylinder length="0.03" radius="0.07" />
             </geometry>
         </collision>
-        <xacro:inertial_cylinder mass="0.1" length="0.05" radius="0.05">
+        <xacro:inertial_cylinder mass="0.1" length="0.03" radius="0.07">
             <origin xyz="0 0 0" rpy="0 0 0"/>
         </xacro:inertial_cylinder>
@@ -114,15 +106,8 @@
         <material>Gazebo/Red</material>
     </gazebo>
-    <!-- BACK LEFT WHEEL -->
-    <joint name="back_left_wheel_joint" type="continuous">
-        <parent link="base_link"/>
-        <child link="back_left_wheel"/>
-        <origin xyz="-0.1 0.175 0" rpy="-${pi/2} 0 0"/>
-        <axis xyz="0 0 1"/>
-    </joint>
     <link name="back_left_wheel">
         <visual>
             <geometry>
-                <cylinder length="0.04" radius="0.05" />
+                <cylinder length="0.03" radius="0.07" />
             </geometry>
             <material name="orange"/>
@@ -130,8 +115,8 @@
         <collision>
             <geometry>
-                <cylinder length="0.04" radius="0.05" />
+                <cylinder length="0.03" radius="0.07" />
             </geometry>
         </collision>
-        <xacro:inertial_cylinder mass="0.1" length="0.05" radius="0.05">
+        <xacro:inertial_cylinder mass="0.1" length="0.03" radius="0.07">
             <origin xyz="0 0 0" rpy="0 0 0"/>
         </xacro:inertial_cylinder>
@@ -140,15 +125,8 @@
         <material>Gazebo/Orange</material>
     </gazebo>
-    <!-- BACK RIGHT WHEEL -->
-    <joint name="back_right_wheel_joint" type="continuous">
-        <parent link="base_link"/>
-        <child link="back_right_wheel"/>
-        <origin xyz="-0.1 -0.175 0" rpy="${pi/2} 0 0"/>
-        <axis xyz="0 0 -1"/>
-    </joint>
     <link name="back_right_wheel">
         <visual>
             <geometry>
-                <cylinder length="0.04" radius="0.05" />
+                <cylinder length="0.03" radius="0.07" />
             </geometry>
             <material name="green"/>
@@ -156,8 +134,8 @@
         <collision>
             <geometry>
-                <cylinder length="0.04" radius="0.05" />
+                <cylinder length="0.03" radius="0.07" />
             </geometry>
         </collision>
-        <xacro:inertial_cylinder mass="0.1" length="0.05" radius="0.05">
+        <xacro:inertial_cylinder mass="0.1" length="0.03" radius="0.07">
             <origin xyz="0 0 0" rpy="0 0 0"/>
         </xacro:inertial_cylinder>
@@ -166,3 +144,32 @@
         <material>Gazebo/Green</material>
     </gazebo>
+    <!-- Wheel Joint -->
+    <!-- FRONT LEFT WHEEL -->
+    <joint name="front_left_wheel_joint" type="continuous">
+        <parent link="base_link"/>
+        <child link="front_left_wheel"/>
+        <origin xyz="0.165 0.205 0" rpy="-${pi/2} 0 0"/>
+        <axis xyz="0 0 1"/>
+    </joint>
+    <!-- FRONT RIGHT WHEEL -->
+    <joint name="front_right_wheel_joint" type="continuous">
+        <parent link="base_link"/>
+        <child link="front_right_wheel"/>
+        <origin xyz="0.165 -0.205 0" rpy="${pi/2} 0 0"/>
+        <axis xyz="0 0 -1"/>
+    </joint>
+    <!-- BACK LEFT WHEEL -->
+    <joint name="back_left_wheel_joint" type="continuous">
+        <parent link="base_link"/>
+        <child link="back_left_wheel"/>
+        <origin xyz="-0.165 0.205 0" rpy="-${pi/2} 0 0"/>
+        <axis xyz="0 0 1"/>
+    </joint>
+    <!-- BACK RIGHT WHEEL -->
+    <joint name="back_right_wheel_joint" type="continuous">
+        <parent link="base_link"/>
+        <child link="back_right_wheel"/>
+        <origin xyz="-0.165 -0.205 0" rpy="${pi/2} 0 0"/>
+        <axis xyz="0 0 -1"/>
+    </joint>
 </robot>

Commit message: ???

File: src/articubot_one/description/gazebo_control.xacro (robot description, xacro)
@@ -7,5 +7,5 @@
             <right_joint>back_right_wheel_joint</right_joint>
             <wheel_separation>0.35</wheel_separation>
-            <wheel_diameter>0.1</wheel_diameter>
+            <wheel_diameter>0.14</wheel_diameter>
             <!-- Limits -->
             <max_wheel_torque>200</max_wheel_torque>
@@ -23,5 +23,5 @@
             <right_joint>front_right_wheel_joint</right_joint>
             <wheel_separation>0.35</wheel_separation>
-            <wheel_diameter>0.1</wheel_diameter>
+            <wheel_diameter>0.14</wheel_diameter>
             <!-- Limits -->
             <max_wheel_torque>200</max_wheel_torque>

File: src/articubot_one/description/gripper.xacro (robot description, xacro)
@@ -1,4 +1,4 @@
 <?xml version="1.0"?>
-<robot xmlns:xacro="http://www.ros.org/wiki/xacro">
+<robot xmlns:xacro="http://www.ros.org/wiki/xacro" xmlns="http://www.ros.org/wiki/xacro">
     <!-- Gripper Base -->
     <link name="gripper_base">
@@ -6,5 +6,5 @@
             <origin xyz="0 0 0" rpy="0 0 0"/>
             <geometry>
-                <box size="0.15 0.05 0.05"/>
+                <box size="0.35 0.05 0.05"/>
             </geometry>
             <material name="gray"/>
@@ -12,7 +12,12 @@
         <collision>
             <geometry>
-                <box size="0.15 0.05 0.05"/>
+                <box size="0.35 0.05 0.05"/>
             </geometry>
         </collision>
+        <inertial>
+            <mass value="0.1"/>
+            <origin xyz="0 0 0" rpy="0 0 0"/>
+            <inertia ixx="0.01" ixy="0" ixz="0" iyy="0.01" iyz="0" izz="0.01"/>
+        </inertial>
     </link>
     <!-- Gripper Finger Left -->
@@ -30,4 +35,9 @@
             </geometry>
         </collision>
+        <inertial>
+            <mass value="0.1"/>
+            <origin xyz="0 0 0" rpy="0 0 0"/>
+            <inertia ixx="0.001" ixy="0" ixz="0" iyy="0.001" iyz="0" izz="0.001"/>
+        </inertial>
     </link>
     <!-- Gripper Finger Right -->
@@ -42,14 +52,13 @@
         <collision>
             <geometry>
-                <box size="0.05 0.02 0.02"/>
+                <box size="0.02 0.1 0.02"/>
             </geometry>
         </collision>
+        <inertial>
+            <mass value="0.1"/>
+            <origin xyz="0 0 0" rpy="0 0 0"/>
+            <inertia ixx="0.001" ixy="0" ixz="0" iyy="0.001" iyz="0" izz="0.001"/>
+        </inertial>
     </link>
-    <!-- Gripper Joints -->
-    <joint name="gripper_base_joint" type="fixed">
-        <parent link="chassis"/>
-        <child link="gripper_base"/>
-        <origin xyz="0 0 0.2" rpy="0 0 0"/>
-    </joint>
     <!-- Vertical Movement Joint for Gripper -->
     <joint name="gripper_vertical_joint" type="prismatic">
@@ -59,4 +68,5 @@
         <axis xyz="0 0 1"/>
         <limit effort="10" lower="0" upper="0.13" velocity="0.1"/>
+        <dynamics damping="0.5" friction="0.1"/>
     </joint>
     <!-- Gripper Finger Joints -->
@@ -67,4 +77,5 @@
         <axis xyz="1 0 0"/>
         <limit effort="10" lower="0" upper="0.1" velocity="0.1"/>
+        <dynamics damping="0.5" friction="0.1"/>
     </joint>
     <joint name="gripper_finger_right_joint" type="prismatic">
@@ -74,14 +85,18 @@
         <axis xyz="1 0 0"/>
         <limit effort="10" lower="-0.1" upper="0" velocity="0.1"/>
+        <dynamics damping="0.5" friction="0.1"/>
     </joint>
     <!-- Gazebo Simulation for Gripper -->
     <gazebo reference="gripper_base">
         <material>Gazebo/Gray</material>
+        <gravity>true</gravity>
     </gazebo>
     <gazebo reference="gripper_finger_left">
         <material>Gazebo/Orange</material>
+        <gravity>true</gravity>
     </gazebo>
     <gazebo reference="gripper_finger_right">
         <material>Gazebo/Orange</material>
+        <gravity>true</gravity>
     </gazebo>
 </robot>

File: src/articubot_one/description/lidar.xacro (robot description, xacro)
@@ -4,5 +4,5 @@
         <parent link="chassis"/>
         <child link="laser_frame"/>
-        <origin xyz="0 0 0.215" rpy="0 0 0"/>
+        <origin xyz="0 0 0.236" rpy="0 0 0"/>
     </joint>
     <link name="laser_frame">

File: src/articubot_one/description/robot_core.xacro (robot description, xacro)
@@ -46,5 +46,5 @@
             <origin xyz="0 0 0.13" rpy="0 0 0"/>
             <geometry>
-                <box size="0.451 0.451 0.15"/>
+                <box size="0.451 0.451 0.18"/>
                 <!-- Hole geometry -->
                 <cylinder length="0.15" radius="0.075"/>
@@ -55,10 +55,10 @@
             <origin xyz="0 0 0.13" rpy="0 0 0"/>
             <geometry>
-                <box size="0.451 0.451 0.15"/>
+                <box size="0.451 0.451 0.18"/>
                 <!-- Hole geometry -->
                 <cylinder length="0.15" radius="0.075"/>
             </geometry>
         </collision>
-        <xacro:inertial_box mass="0.5" x="0.451" y="0.451" z="0.15">
+        <xacro:inertial_box mass="0.5" x="0.451" y="0.451" z="0.18">
             <origin xyz="0 0 0.13" rpy="0 0 0"/>
         </xacro:inertial_box>
