Commit message: finish project robo2?

File: src/articubot_one/description/gazebo_control.xacro (robot description, xacro)
@@ -2,25 +2,12 @@
 <robot xmlns:xacro="http://www.ros.org/wiki/xacro">
     <gazebo>
-        <plugin name='back_wheel' filename='libgazebo_ros_diff_drive.so'>
+        <plugin name='diff_drive' filename='libgazebo_ros_diff_drive.so'>
             <!-- Wheel Information -->
+            <num_wheel_pairs>2</num_wheel_pairs>
+            <left_joint>front_left_wheel_joint</left_joint>
+            <right_joint>front_right_wheel_joint</right_joint>
             <left_joint>back_left_wheel_joint</left_joint>
             <right_joint>back_right_wheel_joint</right_joint>
-            <wheel_separation>0.35</wheel_separation>
-            <wheel_diameter>0.14</wheel_diameter>
-            <!-- Limits -->
-            <max_wheel_torque>200</max_wheel_torque>
-            <max_wheel_acceleration>10.0</max_wheel_acceleration>
-            <!-- Output -->
-            <odometry_frame>odom</odometry_frame>
-            <robot_base_frame>base_link</robot_base_frame>
-            <publish_odom>true</publish_odom>
-            <publish_odom_tf>true</publish_odom_tf>
-            <publish_wheel_tf>true</publish_wheel_tf>
-        </plugin>
-        <plugin name='front_wheel' filename='libgazebo_ros_diff_drive.so'>
-            <!-- Wheel Information -->
-            <left_joint>front_left_wheel_joint</left_joint>
-            <right_joint>front_right_wheel_joint</right_joint>
-            <wheel_separation>0.35</wheel_separation>
+            <wheel_separation>0.35z</wheel_separation>
             <wheel_diameter>0.14</wheel_diameter>
             <!-- Limits -->

File: src/articubot_one/description/gripper.xacro (robot description, xacro)
@@ -1,4 +1,4 @@
 <?xml version="1.0"?>
-<robot xmlns:xacro="http://www.ros.org/wiki/xacro" xmlns="http://www.ros.org/wiki/xacro">
+<robot xmlns:xacro="http://www.ros.org/wiki/xacro" >
     <!-- Gripper Base -->
     <link name="gripper_base">
@@ -11,53 +11,104 @@
         </visual>
         <collision>
+            <origin xyz="0 0 0" rpy="0 0 0"/>
             <geometry>
                 <box size="0.35 0.05 0.05"/>
             </geometry>
+            <surface>
+                <friction>
+                    <ode>
+                        <mu>2.0</mu>  <!-- Increase primary friction -->
+                        <mu2>2.0</mu2>  <!-- Increase secondary friction -->
+                    </ode>
+                </friction>
+                <contact>
+                    <ode>
+                        <restitution>0.0</restitution>  <!-- Lower the bounce factor -->
+                        <soft_cfm>0.1</soft_cfm>  <!-- Soft constraint for smooth contact -->
+                        <soft_erp>0.7</soft_erp>  <!-- Error reduction for smoother response -->
+                        <kp>1000.0</kp>  <!-- Reduce excessive force -->
+                        <kd>100.0</kd>  <!-- Damping to prevent sudden jumps -->
+                        <max_vel>0.01</max_vel>
+                    </ode>
+                </contact>
+            </surface>
         </collision>
-        <inertial>
-            <mass value="0.1"/>
+        <xacro:inertial_box mass="0.5" x="0.35" y="0.05" z="0.05" >
             <origin xyz="0 0 0" rpy="0 0 0"/>
-            <inertia ixx="0.01" ixy="0" ixz="0" iyy="0.01" iyz="0" izz="0.01"/>
-        </inertial>
+        </xacro:inertial_box>
     </link>
     <!-- Gripper Finger Left -->
     <link name="gripper_finger_left">
         <visual>
-            <origin xyz="-0.075 0 0" rpy="0 0 0"/>
+            <origin xyz="-0.075 -0.1 0" rpy="0 0 0"/>
             <geometry>
-                <box size="0.02 0.1 0.02"/>
+                <box size="0.0225 0.2 0.05"/>
             </geometry>
             <material name="orange"/>
         </visual>
         <collision>
+            <origin xyz="-0.075 -0.1 0" rpy="0 0 0"/>
             <geometry>
-                <box size="0.02 0.1 0.02"/>
+                <box size="0.0225 0.2 0.1"/>
             </geometry>
+            <surface>
+                <friction>
+                    <ode>
+                        <mu>2.0</mu>  <!-- Increase primary friction -->
+                        <mu2>2.0</mu2>  <!-- Increase secondary friction -->
+                    </ode>
+                </friction>
+                <contact>
+                    <ode>
+                        <restitution>0.0</restitution>  <!-- Lower the bounce factor -->
+                        <soft_cfm>0.1</soft_cfm>  <!-- Soft constraint for smooth contact -->
+                        <soft_erp>0.7</soft_erp>  <!-- Error reduction for smoother response -->
+                        <kp>1000.0</kp>  <!-- Reduce excessive force -->
+                        <kd>100.0</kd>  <!-- Damping to prevent sudden jumps -->
+                        <max_vel>0.01</max_vel>
+                    </ode>
+                </contact>
+            </surface>
         </collision>
-        <inertial>
-            <mass value="0.1"/>
-            <origin xyz="0 0 0" rpy="0 0 0"/>
-            <inertia ixx="0.001" ixy="0" ixz="0" iyy="0.001" iyz="0" izz="0.001"/>
-        </inertial>
+        <xacro:inertial_box mass="0.3" x="0.0225" y="0.2" z="0.05" >
+            <origin xyz="-0.075 -0.1 0" rpy="0 0 0"/>
+        </xacro:inertial_box>
     </link>
     <!-- Gripper Finger Right -->
     <link name="gripper_finger_right">
         <visual>
-            <origin xyz="0.075 0 0" rpy="0 0 0"/>
+            <origin xyz="0.075 -0.10 0" rpy="0 0 0"/>
             <geometry>
-                <box size="0.02 0.1 0.02"/>
+                <box size="0.0225 0.2 0.05"/>
             </geometry>
             <material name="orange"/>
         </visual>
         <collision>
+            <origin xyz="0.075 -0.10 0" rpy="0 0 0"/>
             <geometry>
-                <box size="0.02 0.1 0.02"/>
+                <box size="0.0225 0.2 0.1"/>
             </geometry>
+            <surface>
+                <friction>
+                    <ode>
+                        <mu>2.0</mu>  <!-- Increase primary friction -->
+                        <mu2>2.0</mu2>  <!-- Increase secondary friction -->
+                    </ode>
+                </friction>
+                <contact>
+                    <ode>
+                        <restitution>0.0</restitution>  <!-- Lower the bounce factor -->
+                        <soft_cfm>0.1</soft_cfm>  <!-- Soft constraint for smooth contact -->
+                        <soft_erp>0.7</soft_erp>  <!-- Error reduction for smoother response -->
+                        <kp>1000.0</kp>  <!-- Reduce excessive force -->
+                        <kd>100.0</kd>  <!-- Damping to prevent sudden jumps -->
+                        <max_vel>0.01</max_vel>
+                    </ode>
+                </contact>
+            </surface>
         </collision>
-        <inertial>
-            <mass value="0.1"/>
-            <origin xyz="0 0 0" rpy="0 0 0"/>
-            <inertia ixx="0.001" ixy="0" ixz="0" iyy="0.001" iyz="0" izz="0.001"/>
-        </inertial>
+        <xacro:inertial_box mass="0.3" x="0.0225" y="0.2" z="0.05" >
+            <origin xyz="0.075 -0.10 0" rpy="0 0 0"/>
+        </xacro:inertial_box>
     </link>
     <!-- Vertical Movement Joint for Gripper -->
@@ -65,8 +116,8 @@
         <parent link="chassis"/>
         <child link="gripper_base"/>
-        <origin xyz="0.25 0 0.05" rpy="0 0 1.57"/>
+        <origin xyz="0.25 0 0" rpy="0 0 1.57"/>
         <axis xyz="0 0 1"/>
-        <limit effort="10" lower="0" upper="0.13" velocity="0.1"/>
-        <dynamics damping="0.5" friction="0.1"/>
+        <limit effort="80" lower="0" upper="0.13" velocity="0.1"/>
+        <dynamics damping="50.0" friction="1.0"/>
     </joint>
     <!-- Gripper Finger Joints -->
@@ -74,16 +125,16 @@
         <parent link="gripper_base"/>
         <child link="gripper_finger_left"/>
-        <origin xyz="-0.075 -0.1 0" rpy="0 0 0"/>
+        <origin xyz="-0.075 0 0" rpy="0 0 0"/>
         <axis xyz="1 0 0"/>
-        <limit effort="10" lower="0" upper="0.1" velocity="0.1"/>
-        <dynamics damping="0.5" friction="0.1"/>
+        <limit effort="100" lower="0" upper="0.1" velocity="0.1"/>
+        <dynamics damping="20.0" friction="1.0"/>
     </joint>
     <joint name="gripper_finger_right_joint" type="prismatic">
         <parent link="gripper_base"/>
         <child link="gripper_finger_right"/>
-        <origin xyz="0.075 -0.1 0" rpy="0 0 0"/>
+        <origin xyz="0.075 0 0" rpy="0 0 0"/>
         <axis xyz="1 0 0"/>
-        <limit effort="10" lower="-0.1" upper="0" velocity="0.1"/>
-        <dynamics damping="0.5" friction="0.1"/>
+        <limit effort="100" lower="-0.1" upper="0" velocity="0.1"/>
+        <dynamics damping="20.0" friction="1.0"/>
     </joint>
     <!-- Gazebo Simulation for Gripper -->
@@ -91,12 +142,32 @@
         <material>Gazebo/Gray</material>
         <gravity>true</gravity>
+        <ode>
+            <solver_iterations>500</solver_iterations>  <!-- Increase solver iterations -->
+            <solver_type>quick_nonlinear</solver_type>  <!-- Adjust solver for stability -->
+        </ode>
     </gazebo>
     <gazebo reference="gripper_finger_left">
         <material>Gazebo/Orange</material>
         <gravity>true</gravity>
+        <ode>
+            <solver_iterations>500</solver_iterations>  <!-- Increase solver iterations -->
+            <solver_type>quick_nonlinear</solver_type>  <!-- Adjust solver for stability -->
+        </ode>
+        <!-- <plugin name="gazebo_gripper" filename="libgazebo_ros_vacuum_gripper.so">
+            <always_on>true</always_on>
+            <topic>gripper/grasp</topic>
+        </plugin> -->
     </gazebo>
     <gazebo reference="gripper_finger_right">
         <material>Gazebo/Orange</material>
         <gravity>true</gravity>
+        <ode>
+            <solver_iterations>500</solver_iterations>  <!-- Increase solver iterations -->
+            <solver_type>quick_nonlinear</solver_type>  <!-- Adjust solver for stability -->
+        </ode>
+        <!-- <plugin name="gazebo_gripper" filename="libgazebo_ros_vacuum_gripper.so">
+            <always_on>true</always_on>
+            <topic>gripper/grasp</topic>
+        </plugin> -->
     </gazebo>
 </robot>

File: src/articubot_one/description/robot.urdf.xacro (robot description, xacro)
@@ -8,3 +8,17 @@
     <xacro:include filename="lidar.xacro" />
     <xacro:include filename="gripper.xacro" />
+    <xacro:include filename="gripper_vertical_tranmission.xacro" />
+    <xacro:include filename="gripper_finger_left_tranmission.xacro" />
+    <xacro:include filename="gripper_finger_right_tranmission.xacro" />
+    <xacro:include filename="robot_control.urdf.xacro"/>
+    <!-- <xacro:include filename="redbox150mm.xacro"/> -->
+    <xacro:robot_controller/>
+    <ros2_control name="gripper_robot_gazebo_system" type="system">
+        <hardware>
+            <plugin>gazebo_ros2_control/GazeboSystem</plugin>
+        </hardware>
+        <xacro:gripper_vertical_tranmission/>
+        <xacro:gripper_finger_left_tranmission/>
+        <xacro:gripper_finger_right_tranmission/>
+    </ros2_control>
 </robot>

File: src/articubot_one/description/robot_core.xacro (robot description, xacro)
@@ -60,5 +60,5 @@
             </geometry>
         </collision>
-        <xacro:inertial_box mass="0.5" x="0.451" y="0.451" z="0.18">
+        <xacro:inertial_box mass="200" x="0.451" y="0.451" z="0.18">
             <origin xyz="0 0 0.13" rpy="0 0 0"/>
         </xacro:inertial_box>
@@ -80,5 +80,5 @@
             </geometry>
         </collision>
-        <xacro:inertial_cylinder mass="0.1" length="0.03" radius="0.07">
+        <xacro:inertial_cylinder mass="20" length="0.03" radius="0.07">
             <origin xyz="0 0 0" rpy="0 0 0"/>
         </xacro:inertial_cylinder>
@@ -99,5 +99,5 @@
             </geometry>
         </collision>
-        <xacro:inertial_cylinder mass="0.1" length="0.03" radius="0.07">
+        <xacro:inertial_cylinder mass="20" length="0.03" radius="0.07">
             <origin xyz="0 0 0" rpy="0 0 0"/>
         </xacro:inertial_cylinder>
@@ -118,5 +118,5 @@
             </geometry>
         </collision>
-        <xacro:inertial_cylinder mass="0.1" length="0.03" radius="0.07">
+        <xacro:inertial_cylinder mass="20" length="0.03" radius="0.07">
             <origin xyz="0 0 0" rpy="0 0 0"/>
         </xacro:inertial_cylinder>
@@ -137,5 +137,5 @@
             </geometry>
         </collision>
-        <xacro:inertial_cylinder mass="0.1" length="0.03" radius="0.07">
+        <xacro:inertial_cylinder mass="20" length="0.03" radius="0.07">
             <origin xyz="0 0 0" rpy="0 0 0"/>
         </xacro:inertial_cylinder>
