Commit message: update xacro file

File: src/articubot_one/description/gripper_tranmission.xacro (robot description, xacro)
@@ -1,23 +1,33 @@
 <?xml version="1.0"?>
-<robot xmlns:xacro="http://www.ros.org/wiki/xacro">
-    <xacro:macro name="gripper_transmission" params="">
-        <transmission name="gripper_trans">
-            <type>transmission_interface/SimpleTransmission</type>
-            <joint name="gripper_vertical_joint">
-                <command_interface name="position" />
-                <state_interface name="position" />
-                <state_interface name="velocity" />
-            </joint>
-            <joint name="gripper_finger_left_joint">
-                <command_interface name="position" />
-                <state_interface name="position" />
-                <state_interface name="velocity" />
-            </joint>
-            <joint name="gripper_finger_right_joint">
-                <command_interface name="position" />
-                <state_interface name="position" />
-                <state_interface name="velocity" />
-            </joint>
-        </transmission>
+<robot xmlns:xacro="http://ros.org/wiki/xacro">
+    <xacro:macro name="gripper_finger_left_tranmission" params="">
+        <joint name="gripper_finger_left_joint">
+            <command_interface name="velocity">
+                <param name="min">0</param>
+                <param name="max">0.1</param>
+            </command_interface>
+            <state_interface name="position" />
+            <state_interface name="velocity" />
+        </joint>
+    </xacro:macro>
+    <xacro:macro name="gripper_finger_right_tranmission" params="">
+        <joint name="gripper_finger_right_joint">
+            <command_interface name="velocity">
+                <param name="min">-0.1</param>
+                <param name="max">0</param>
+            </command_interface>
+            <state_interface name="position" />
+            <state_interface name="velocity" />
+        </joint>
+    </xacro:macro>
+    <xacro:macro name="gripper_vertical_tranmission" params="">
+        <joint name="gripper_vertical_joint">
+            <command_interface name="velocity">
+                <param name="min">0</param>
+                <param name="max">0.13</param>
+            </command_interface>
+            <state_interface name="position" />
+            <state_interface name="velocity" />
+        </joint>
     </xacro:macro>
 </robot>

File: src/articubot_one/description/robot.urdf.xacro (robot description, xacro)
@@ -8,8 +8,6 @@
     <xacro:include filename="lidar.xacro" />
     <xacro:include filename="gripper.xacro" />
-    <xacro:include filename="gripper_vertical_tranmission.xacro" />
-    <xacro:include filename="gripper_finger_left_tranmission.xacro" />
-    <xacro:include filename="gripper_finger_right_tranmission.xacro" />
-    <xacro:include filename="robot_control.urdf.xacro"/>
+    <xacro:include filename="gripper_tranmission.xacro" />
+    <xacro:include filename="gazebo_plugin.xacro"/>
     <!-- <xacro:include filename="redbox150mm.xacro"/> -->
     <xacro:robot_controller/>
